Commit message: feat:修改 urdf 文件

File: urdf_tutorial/urdf/beacon.urdf (robot description, URDF)
Before this commit: robot beacon, 2 links, 1 joints
Links:
- link laser_link: geometry visual cylinder length=0.6 radius=0.6

Commit message: feat: 迁移了一个其它机器人的框架

File: urdf_tutorial/urdf/beacon.urdf (robot description, URDF)
Before this commit: robot beacon, 2 links, 1 joints
Links:
- removed link laser_link
- added link box, mass 1; collision box size=0.08 0.08 0.08; visual box size=0.08 0.08 0.08
- added link gripper_pole, mass 0.05; collision cylinder length=0.2 radius=0.01; visual cylinder length=0.2 radius=0.01
- added link head, mass 2; collision sphere radius=0.2; visual sphere radius=0.2
- added link left_back_wheel, mass 1; collision cylinder length=0.1 radius=0.035; visual cylinder length=0.1 radius=0.035
- added link left_base, mass 10; collision box size=0.4 0.1 0.1; visual box size=0.4 0.1 0.1
- added link left_front_wheel, mass 1; collision cylinder length=0.1 radius=0.035; visual cylinder length=0.1 radius=0.035
- added link left_gripper, mass 0.05; collision mesh filename=package://urdf_tutorial/meshes/l_finger.dae; visual mesh filename=package://urdf_tutorial/meshes/l_finger.dae
- added link left_leg, mass 10; collision box size=0.6 0.1 0.2; visual box size=0.6 0.1 0.2
- added link left_tip, mass 0.05; collision mesh filename=package://urdf_tutorial/meshes/l_finger_tip.dae; visual mesh filename=package://urdf_tutorial/meshes/l_finger_tip.dae
- added link right_back_wheel, mass 1; collision cylinder length=0.1 radius=0.035; visual cylinder length=0.1 radius=0.035
- added link right_base, mass 10; collision box size=0.4 0.1 0.1; visual box size=0.4 0.1 0.1
- added link right_front_wheel, mass 1; collision cylinder length=0.1 radius=0.035; visual cylinder length=0.1 radius=0.035
- added link right_gripper, mass 0.05; collision mesh filename=package://urdf_tutorial/meshes/l_finger.dae; visual mesh filename=package://urdf_tutorial/meshes/l_finger.dae
- added link right_leg, mass 10; collision box size=0.6 0.1 0.2; visual box size=0.6 0.1 0.2
- added link right_tip, mass 0.05; collision mesh filename=package://urdf_tutorial/meshes/l_finger_tip.dae; visual mesh filename=package://urdf_tutorial/meshes/l_finger_tip.dae
- link base_link: mass None -> 10; geometry collision cylinder length=0.6 radius=0.2; visual cylinder length=0.6 radius=0.2
Joints:
- removed joint laser_joint
- added joint base_to_left_leg: type fixed, parent base_link, child left_leg, origin xyz=0 0.22 0.25
- added joint base_to_right_leg: type fixed, parent base_link, child right_leg, origin xyz=0 -0.22 0.25
- added joint gripper_extension: type prismatic, parent base_link, child gripper_pole, origin xyz=0.19 0 0.2 rpy=0 0 0, limit lower=-0.38 upper=0 effort=1000.0 velocity=0.5
- added joint head_swivel: type continuous, parent base_link, child head, origin xyz=0 0 0.3, axis 0 0 1
- added joint left_back_wheel_joint: type continuous, parent left_base, child left_back_wheel, origin xyz=-0.133333333333 0 -0.085 rpy=0 0 0, axis 0 1 0
- added joint left_base_joint: type fixed, parent left_leg, child left_base, origin xyz=0 0 -0.6
- added joint left_front_wheel_joint: type continuous, parent left_base, child left_front_wheel, origin xyz=0.133333333333 0 -0.085 rpy=0 0 0, axis 0 1 0
- added joint left_gripper_joint: type revolute, parent gripper_pole, child left_gripper, origin xyz=0.2 0.01 0 rpy=0 0 0, axis 0 0 1, limit lower=0.0 upper=0.548 effort=1000.0 velocity=0.5
- added joint left_tip_joint: type fixed, parent left_gripper, child left_tip
- added joint right_back_wheel_joint: type continuous, parent right_base, child right_back_wheel, origin xyz=-0.133333333333 0 -0.085 rpy=0 0 0, axis 0 1 0
- added joint right_base_joint: type fixed, parent right_leg, child right_base, origin xyz=0 0 -0.6
- added joint right_front_wheel_joint: type continuous, parent right_base, child right_front_wheel, origin xyz=0.133333333333 0 -0.085 rpy=0 0 0, axis 0 1 0
- added joint right_gripper_joint: type revolute, parent gripper_pole, child right_gripper, origin xyz=0.2 -0.01 0 rpy=0 0 0, axis 0 0 -1, limit lower=0.0 upper=0.548 effort=1000.0 velocity=0.5
- added joint right_tip_joint: type fixed, parent right_gripper, child right_tip
- added joint tobox: type fixed, parent head, child box, origin xyz=0.1814 0 0.1414

Commit message: feat:修改 beacon 的模型为一个小车

File: urdf_tutorial/urdf/beacon.urdf (robot description, URDF)
Before this commit: robot physics, 16 links, 15 joints
Links:
- removed link box
- removed link gripper_pole
- removed link head
- removed link left_back_wheel
- removed link left_base
- removed link left_front_wheel
- removed link left_gripper
- removed link left_leg
- removed link left_tip
- removed link right_back_wheel
- removed link right_base
- removed link right_front_wheel
- removed link right_gripper
- removed link right_leg
- removed link right_tip
- added link base_footprint
- added link base_scan, mass 0.114; collision cylinder length=0.0315 radius=0.055; visual mesh filename=package://urdf_tutorial/meshes/turtlebot3/sensors/lds.stl scale=0.001 0.001 0.001
- added link camera_depth_frame
- added link camera_depth_optical_frame
- added link camera_link; collision box size=0.012 0.132 0.020; visual mesh filename=package://urdf_tutorial/meshes/turtlebot3/sensors/r200.dae
- added link camera_rgb_frame
- added link camera_rgb_optical_frame
- added link caster_back_left_link, mass 0.005; collision box size=0.030 0.009 0.020
- added link caster_back_right_link, mass 0.005; collision box size=0.030 0.009 0.020
- added link imu_link
- added link wheel_left_link, mass 2.8498940e-02; collision cylinder length=0.018 radius=0.033; visual mesh filename=package://urdf_tutorial/meshes/turtlebot3/wheels/left_tire.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 scale=0.001 0.001 0.001
- added link wheel_right_link, mass 2.8498940e-02; collision cylinder length=0.018 radius=0.033; visual mesh filename=package://urdf_tutorial/meshes/turtlebot3/wheels/right_tire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 scale=0.001 0.001 0.001
- link base_link: mass 10 -> 1.3729096e+00; geometry collision box size=0.266 0.266 0.094; visual mesh filename=package://urdf_tutorial/meshes/turtlebot3/bases/waffle_base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 scale=0.001 0.001 0.001
Joints:
- removed joint base_to_left_leg
- removed joint base_to_right_leg
- removed joint gripper_extension
- removed joint head_swivel
- removed joint left_back_wheel_joint
- removed joint left_base_joint
- removed joint left_front_wheel_joint
- removed joint left_gripper_joint
- removed joint left_tip_joint
- removed joint right_back_wheel_joint
- removed joint right_base_joint
- removed joint right_front_wheel_joint
- removed joint right_gripper_joint
- removed joint right_tip_joint
- removed joint tobox
- added joint base_joint: type fixed, parent base_footprint, child base_link, origin xyz=0 0 0.010 rpy=0 0 0
- added joint camera_depth_joint: type fixed, parent camera_link, child camera_depth_frame, origin xyz=${r200_cam_rgb_px} ${r200_cam_rgb_py + r200_cam_depth_offset} ${r200_cam_rgb_pz} rpy=0 0 0
- added joint camera_depth_optical_joint: type fixed, parent camera_depth_frame, child camera_depth_optical_frame, origin xyz=0 0 0 rpy=-1.57 0 -1.57
- added joint camera_joint: type fixed, parent base_link, child camera_link, origin xyz=0.064 -0.065 0.094 rpy=0 0 0
- added joint camera_rgb_joint: type fixed, parent camera_link, child camera_rgb_frame, origin xyz=${r200_cam_rgb_px} ${r200_cam_rgb_py} ${r200_cam_rgb_pz} rpy=0 0 0
- added joint camera_rgb_optical_joint: type fixed, parent camera_rgb_frame, child camera_rgb_optical_frame, origin xyz=0 0 0 rpy=-1.57 0 -1.57
- added joint caster_back_left_joint: type fixed, parent base_link, child caster_back_left_link, origin xyz=-0.177 0.064 -0.004 rpy=-1.57 0 0
- added joint caster_back_right_joint: type fixed, parent base_link, child caster_back_right_link, origin xyz=-0.177 -0.064 -0.004 rpy=-1.57 0 0
- added joint imu_joint: type fixed, parent base_link, child imu_link, origin xyz=0.0 0 0.068 rpy=0 0 0
- added joint scan_joint: type fixed, parent base_link, child base_scan, origin xyz=-0.064 0 0.122 rpy=0 0 0
- added joint wheel_left_joint: type continuous, parent base_link, child wheel_left_link, origin xyz=0.0 0.144 0.023 rpy=-1.57 0 0, axis 0 0 1
- added joint wheel_right_joint: type continuous, parent base_link, child wheel_right_link, origin xyz=0.0 -0.144 0.023 rpy=-1.57 0 0, axis 0 0 1
