Commit message: feat:添加 xacro，使用 xacro 生成 urdf

File: urdf_tutorial/urdf/beacon.urdf.xacro (robot description, xacro)
@@ -1,17 +1,17 @@
 <?xml version="1.0" ?>
-<!-- =================================================================================== -->
-<!-- |    This document was autogenerated by xacro from src/ros2_tutorial/urdf_tutorial/urdf/beacon.urdf.xacro | -->
-<!-- |    EDITING THIS FILE BY HAND IS NOT RECOMMENDED                                 | -->
-<!-- =================================================================================== -->
-<robot name="turtlebot3_waffle">
+<robot name="turtlebot3_waffle" xmlns:xacro="http://ros.org/wiki/xacro">
+  <xacro:property name="r200_cam_rgb_px" value="0.005"/>
+  <xacro:property name="r200_cam_rgb_py" value="0.018"/>
+  <xacro:property name="r200_cam_rgb_pz" value="0.013"/>
+  <xacro:property name="r200_cam_depth_offset" value="0.01"/>
   <link name="base_footprint"/>
   <joint name="base_joint" type="fixed">
     <parent link="base_footprint"/>
-    <child link="base_link"/>
-    <origin rpy="0 0 0" xyz="0 0 0.010"/>
+    <child link="base_link" />
+    <origin xyz="0 0 0.010" rpy="0 0 0"/>
   </joint>
   <link name="base_link">
     <visual>
-      <origin rpy="0 0 0" xyz="-0.064 0 0.0"/>
+      <origin xyz="-0.064 0 0.0" rpy="0 0 0"/>
       <geometry>
         <mesh filename="package://urdf_tutorial/meshes/turtlebot3/bases/waffle_base.stl" scale="0.001 0.001 0.001"/>
@@ -22,5 +22,5 @@
     </visual>
     <collision>
-      <origin rpy="0 0 0" xyz="-0.064 0 0.047"/>
+      <origin xyz="-0.064 0 0.047" rpy="0 0 0"/>
       <geometry>
         <box size="0.266 0.266 0.094"/>
@@ -28,7 +28,9 @@
     </collision>
     <inertial>
-      <origin rpy="0 0 0" xyz="0 0 0"/>
+      <origin xyz="0 0 0" rpy="0 0 0"/>
       <mass value="1.3729096e+00"/>
-      <inertia ixx="8.7002718e-03" ixy="-4.7576583e-05" ixz="1.1160499e-04" iyy="8.6195418e-03" iyz="-3.5422299e-06" izz="1.4612727e-02"/>
+      <inertia ixx="8.7002718e-03" ixy="-4.7576583e-05" ixz="1.1160499e-04"
+               iyy="8.6195418e-03" iyz="-3.5422299e-06"
+               izz="1.4612727e-02" />
     </inertial>
   </link>
@@ -36,10 +38,10 @@
     <parent link="base_link"/>
     <child link="wheel_left_link"/>
-    <origin rpy="-1.57 0 0" xyz="0.0 0.144 0.023"/>
+    <origin xyz="0.0 0.144 0.023" rpy="-1.57 0 0"/>
     <axis xyz="0 0 1"/>
   </joint>
   <link name="wheel_left_link">
     <visual>
-      <origin rpy="1.57 0 0" xyz="0 0 0"/>
+      <origin xyz="0 0 0" rpy="1.57 0 0"/>
       <geometry>
         <mesh filename="package://urdf_tutorial/meshes/turtlebot3/wheels/left_tire.stl" scale="0.001 0.001 0.001"/>
@@ -50,5 +52,5 @@
     </visual>
     <collision>
-      <origin rpy="0 0 0" xyz="0 0 0"/>
+      <origin xyz="0 0 0" rpy="0 0 0"/>
       <geometry>
         <cylinder length="0.018" radius="0.033"/>
@@ -56,18 +58,20 @@
     </collision>
     <inertial>
-      <origin xyz="0 0 0"/>
-      <mass value="2.8498940e-02"/>
-      <inertia ixx="1.1175580e-05" ixy="-4.2369783e-11" ixz="-5.9381719e-09" iyy="1.1192413e-05" iyz="-1.4400107e-11" izz="2.0712558e-05"/>
-    </inertial>
+      <origin xyz="0 0 0" />
+      <mass value="2.8498940e-02" />
+      <inertia ixx="1.1175580e-05" ixy="-4.2369783e-11" ixz="-5.9381719e-09"
+               iyy="1.1192413e-05" iyz="-1.4400107e-11"
+               izz="2.0712558e-05" />
+      </inertial>
   </link>
   <joint name="wheel_right_joint" type="continuous">
     <parent link="base_link"/>
     <child link="wheel_right_link"/>
-    <origin rpy="-1.57 0 0" xyz="0.0 -0.144 0.023"/>
+    <origin xyz="0.0 -0.144 0.023" rpy="-1.57 0 0"/>
     <axis xyz="0 0 1"/>
   </joint>
   <link name="wheel_right_link">
     <visual>
-      <origin rpy="1.57 0 0" xyz="0 0 0"/>
+      <origin xyz="0 0 0" rpy="1.57 0 0"/>
       <geometry>
         <mesh filename="package://urdf_tutorial/meshes/turtlebot3/wheels/right_tire.stl" scale="0.001 0.001 0.001"/>
@@ -78,5 +82,5 @@
     </visual>
     <collision>
-      <origin rpy="0 0 0" xyz="0 0 0"/>
+      <origin xyz="0 0 0" rpy="0 0 0"/>
       <geometry>
         <cylinder length="0.018" radius="0.033"/>
@@ -84,17 +88,19 @@
     </collision>
     <inertial>
-      <origin xyz="0 0 0"/>
-      <mass value="2.8498940e-02"/>
-      <inertia ixx="1.1175580e-05" ixy="-4.2369783e-11" ixz="-5.9381719e-09" iyy="1.1192413e-05" iyz="-1.4400107e-11" izz="2.0712558e-05"/>
-    </inertial>
+      <origin xyz="0 0 0" />
+      <mass value="2.8498940e-02" />
+      <inertia ixx="1.1175580e-05" ixy="-4.2369783e-11" ixz="-5.9381719e-09"
+               iyy="1.1192413e-05" iyz="-1.4400107e-11"
+               izz="2.0712558e-05" />
+      </inertial>
   </link>
   <joint name="caster_back_right_joint" type="fixed">
     <parent link="base_link"/>
     <child link="caster_back_right_link"/>
-    <origin rpy="-1.57 0 0" xyz="-0.177 -0.064 -0.004"/>
+    <origin xyz="-0.177 -0.064 -0.004" rpy="-1.57 0 0"/>
   </joint>
   <link name="caster_back_right_link">
     <collision>
-      <origin rpy="0 0 0" xyz="0 0.001 0"/>
+      <origin xyz="0 0.001 0" rpy="0 0 0"/>
       <geometry>
         <box size="0.030 0.009 0.020"/>
@@ -102,7 +108,9 @@
     </collision>
     <inertial>
-      <origin xyz="0 0 0"/>
-      <mass value="0.005"/>
-      <inertia ixx="0.001" ixy="0.0" ixz="0.0" iyy="0.001" iyz="0.0" izz="0.001"/>
+      <origin xyz="0 0 0" />
+      <mass value="0.005" />
+      <inertia ixx="0.001" ixy="0.0" ixz="0.0"
+               iyy="0.001" iyz="0.0"
+               izz="0.001" />
     </inertial>
   </link>
@@ -110,9 +118,9 @@
     <parent link="base_link"/>
     <child link="caster_back_left_link"/>
-    <origin rpy="-1.57 0 0" xyz="-0.177 0.064 -0.004"/>
+    <origin xyz="-0.177 0.064 -0.004" rpy="-1.57 0 0"/>
   </joint>
   <link name="caster_back_left_link">
     <collision>
-      <origin rpy="0 0 0" xyz="0 0.001 0"/>
+      <origin xyz="0 0.001 0" rpy="0 0 0"/>
       <geometry>
         <box size="0.030 0.009 0.020"/>
@@ -120,7 +128,9 @@
     </collision>
     <inertial>
-      <origin xyz="0 0 0"/>
-      <mass value="0.005"/>
-      <inertia ixx="0.001" ixy="0.0" ixz="0.0" iyy="0.001" iyz="0.0" izz="0.001"/>
+      <origin xyz="0 0 0" />
+      <mass value="0.005" />
+      <inertia ixx="0.001" ixy="0.0" ixz="0.0"
+               iyy="0.001" iyz="0.0"
+               izz="0.001" />
     </inertial>
   </link>
@@ -128,5 +138,5 @@
     <parent link="base_link"/>
     <child link="imu_link"/>
-    <origin rpy="0 0 0" xyz="0.0 0 0.068"/>
+    <origin xyz="0.0 0 0.068" rpy="0 0 0"/>
   </joint>
   <link name="imu_link"/>
@@ -134,9 +144,9 @@
     <parent link="base_link"/>
     <child link="base_scan"/>
-    <origin rpy="0 0 0" xyz="-0.064 0 0.122"/>
+    <origin xyz="-0.064 0 0.122" rpy="0 0 0"/>
   </joint>
   <link name="base_scan">
     <visual>
-      <origin rpy="0 0 0" xyz="0 0 0"/>
+      <origin xyz="0 0 0" rpy="0 0 0"/>
       <geometry>
         <mesh filename="package://urdf_tutorial/meshes/turtlebot3/sensors/lds.stl" scale="0.001 0.001 0.001"/>
@@ -147,5 +157,5 @@
     </visual>
     <collision>
-      <origin rpy="0 0 0" xyz="0.015 0 -0.0065"/>
+      <origin xyz="0.015 0 -0.0065" rpy="0 0 0"/>
       <geometry>
         <cylinder length="0.0315" radius="0.055"/>
@@ -153,11 +163,13 @@
     </collision>
     <inertial>
-      <mass value="0.114"/>
-      <origin xyz="0 0 0"/>
-      <inertia ixx="0.001" ixy="0.0" ixz="0.0" iyy="0.001" iyz="0.0" izz="0.001"/>
+      <mass value="0.114" />
+      <origin xyz="0 0 0" />
+      <inertia ixx="0.001" ixy="0.0" ixz="0.0"
+               iyy="0.001" iyz="0.0"
+               izz="0.001" />
     </inertial>
   </link>
   <joint name="camera_joint" type="fixed">
-    <origin rpy="0 0 0" xyz="0.064 -0.065 0.094"/>
+    <origin xyz="0.064 -0.065 0.094" rpy="0 0 0"/>
     <parent link="base_link"/>
     <child link="camera_link"/>
@@ -165,11 +177,11 @@
   <link name="camera_link">
     <visual>
-      <origin rpy="1.57 0 1.57" xyz="0 0 0"/>
-      <geometry>
-        <mesh filename="package://urdf_tutorial/meshes/turtlebot3/sensors/r200.dae"/>
-      </geometry>
-    </visual>
-    <collision>
-      <origin rpy="0 0 0" xyz="0.003 0.065 0.007"/>
+     <origin xyz="0 0 0" rpy="1.57 0 1.57"/>
+      <geometry>
+       <mesh filename="package://urdf_tutorial/meshes/turtlebot3/sensors/r200.dae" />
+      </geometry>
+    </visual>
+    <collision>
+      <origin xyz="0.003 0.065 0.007" rpy="0 0 0"/>
       <geometry>
         <box size="0.012 0.132 0.020"/>
@@ -177,5 +189,5 @@
     </collision>
     <!-- This inertial field needs doesn't contain reliable data!! -->
-    <!--   <inertial>
+<!--   <inertial>
       <mass value="0.564" />
       <origin xyz="0 0 0" />
@@ -186,5 +198,5 @@
   </link>
   <joint name="camera_rgb_joint" type="fixed">
-    <origin rpy="0 0 0" xyz="0.005 0.018 0.013"/>
+    <origin xyz="${r200_cam_rgb_px} ${r200_cam_rgb_py} ${r200_cam_rgb_pz}" rpy="0 0 0"/>
     <parent link="camera_link"/>
     <child link="camera_rgb_frame"/>
@@ -192,5 +204,5 @@
   <link name="camera_rgb_frame"/>
   <joint name="camera_rgb_optical_joint" type="fixed">
-    <origin rpy="-1.57 0 -1.57" xyz="0 0 0"/>
+    <origin xyz="0 0 0" rpy="-1.57 0 -1.57"/>
     <parent link="camera_rgb_frame"/>
     <child link="camera_rgb_optical_frame"/>
@@ -198,5 +210,5 @@
   <link name="camera_rgb_optical_frame"/>
   <joint name="camera_depth_joint" type="fixed">
-    <origin rpy="0 0 0" xyz="0.005 0.027999999999999997 0.013"/>
+    <origin xyz="${r200_cam_rgb_px} ${r200_cam_rgb_py + r200_cam_depth_offset} ${r200_cam_rgb_pz}" rpy="0 0 0"/>
     <parent link="camera_link"/>
     <child link="camera_depth_frame"/>
@@ -204,5 +216,5 @@
   <link name="camera_depth_frame"/>
   <joint name="camera_depth_optical_joint" type="fixed">
-    <origin rpy="-1.57 0 -1.57" xyz="0 0 0"/>
+    <origin xyz="0 0 0" rpy="-1.57 0 -1.57"/>
     <parent link="camera_depth_frame"/>
     <child link="camera_depth_optical_frame"/>
