Commit message: feat:查看urdf中主要标签 visual collision inertial 的含义
同时查看了相应的子标签以及其它的一些标签

File: src/node_demo/urdf/robot.urdf (robot description, URDF)
Before this commit: robot beaconcar, 5 links, 4 joints
Links:
- added link arm_base
- link base_link: mass None -> 100; geometry collision box size=0.2 .3 0.1; visual box size=0.2 .3 .1

Commit message: feat:beaconbots 更新，添加了一些其他的功能

File: src/node_demo/urdf/robot.urdf (robot description, URDF)
Before this commit: robot beaconcar, 6 links, 4 joints
Links:
- added link arm_button, mass 1; collision box size=0.05 0.05 0.5; visual box size=0.05 0.05 0.5
- added link arm_upper, mass 1; collision box size=0.05 0.05 0.5; visual box size=0.05 0.05 0.5
- added link left_gripper, mass 1; collision box size=0.1 .1 .1; visual mesh filename=package://urdf_tutorial/meshes/l_finger.dae
- added link left_tip, mass 1; visual mesh filename=package://urdf_tutorial/meshes/l_finger_tip.dae
- added link right_gripper, mass 1; collision box size=0.1 .1 .1; visual mesh filename=package://urdf_tutorial/meshes/l_finger.dae
- added link right_tip, mass 1; visual mesh filename=package://urdf_tutorial/meshes/l_finger_tip.dae
- link arm_base: mass None -> 1; geometry collision box size=0.1 .1 .1; visual box size=0.1 0.1 0.1
- link base_link: geometry collision box size=0.2 .3 0.1; visual box size=0.3 .2 .1
Joints:
- added joint arm_button_2_arm_base: type revolute, parent base_link, child arm_button, origin xyz=0 0 0.15, axis 1 0 0, limit lower=-1.0 upper=1.0 effort=1000.0 velocity=0.5
- added joint arm_upper_to_arm_button: type revolute, parent arm_button, child arm_upper, origin xyz=0.0 0 0.45, axis 1 0 0, limit lower=-2.5 upper=2.5 effort=1000.0 velocity=0.5
- added joint base_2_arm_base: type continuous, parent base_link, child arm_base, origin xyz=0 0 0, axis 0 0 1
- added joint left_gripper_2_arm_upper: type revolute, parent arm_upper, child left_gripper, origin xyz=0.06 0 0.4 rpy=0 -1.57 0, axis 0 0 1, limit lower=0. upper=0.548 effort=1000. velocity=0.5
- added joint left_tip_joint: type fixed, parent left_gripper, child left_tip
- added joint right_gripper_2_arm_upper: type revolute, parent arm_upper, child right_gripper, origin xyz=0.06 0 0.4 rpy=0 -1.57 0, axis 0 0 -1, limit lower=0. upper=0.548 effort=1000. velocity=0.5
- added joint right_tip_joint: type fixed, parent right_gripper, child right_tip

Commit message: fix:修复碰撞错误，以及根链接惯性错误

File: src/node_demo/urdf/robot.urdf (robot description, URDF)
Before this commit: robot beaconcar, 12 links, 11 joints
Links:
- added link dummy_link, mass 100.0
- link base_link: mass 100 -> None
- link left_tip: geometry collision box size=0.1 0.1 0.1; visual mesh filename=package://urdf_tutorial/meshes/l_finger_tip.dae
- link right_tip: geometry collision box size=0.1 0.1 0.1; visual mesh filename=package://urdf_tutorial/meshes/l_finger_tip.dae
Joints:
- added joint base_joint: type fixed, parent dummy_link, child base_link
- joint arm_button_2_arm_base: parent base_link -> arm_base

Commit message: feat:更新urdf和rviz让小车的轮子可以转动，以及在rviz中显示

File: src/node_demo/urdf/robot.urdf (robot description, URDF)
Before this commit: robot beaconcar, 13 links, 12 joints
Joints:
- joint base_2_wheel_left_back: axis (none) -> 1 0 0; limit (none) -> lower=-1.0 upper=1.0 effort=1000.0 velocity=0.5; type fixed -> revolute
- joint base_2_wheel_left_front: axis (none) -> 1 0 0; limit (none) -> lower=-1.0 upper=1.0 effort=1000.0 velocity=0.5; type fixed -> revolute
- joint base_2_wheel_right_back: axis (none) -> 1 0 0; limit (none) -> lower=-1.0 upper=1.0 effort=1000.0 velocity=0.5; type fixed -> revolute
- joint base_2_wheel_right_front: axis (none) -> 1 0 0; limit (none) -> lower=-1.0 upper=1.0 effort=1000.0 velocity=0.5; type fixed -> revolute

Commit message: feat:添加关于ros2中如何移动小车，以及twis和join_statetopic的使用

File: src/node_demo/urdf/robot.urdf (robot description, URDF)
Before this commit: robot beaconcar, 13 links, 12 joints
Links:
- removed link dummy_link
- link base_link: mass None -> 100
Joints:
- removed joint base_joint
- joint base_2_wheel_left_back: axis 1 0 0 -> 0 1 0; limit lower=-1.0 upper=1.0 effort=1000.0 velocity=0.5 -> lower=-0.01 upper=0.01 effort=1000.0 velocity=0.5
- joint base_2_wheel_left_front: axis 1 0 0 -> 0 1 0; limit lower=-1.0 upper=1.0 effort=1000.0 velocity=0.5 -> lower=-0.01 upper=0.01 effort=1000.0 velocity=0.5
- joint base_2_wheel_right_back: axis 1 0 0 -> 0 1 0; limit lower=-1.0 upper=1.0 effort=1000.0 velocity=0.5 -> lower=-0.01 upper=0.01 effort=1000.0 velocity=0.5
- joint base_2_wheel_right_front: axis 1 0 0 -> 0 1 0; limit lower=-1.0 upper=1.0 effort=1000.0 velocity=0.5 -> lower=-0.01 upper=0.01 effort=1000.0 velocity=0.5
